File: plusz-end-card-generic/plusz-end-card-generic.kicad_pcb (KiCad board)
At the start: 4 copper layers, 99.8 x 94.6 mm, 28 parts, among them J2 Harwin M55-7101242R, J3 Harwin M55-7101242R, J4 Harwin M55-7101242R, J5 Harwin M55-7101242R

Commit message: new
Parts:
- added G***: LOGO, Foras_Promineo_Github_Local:Sierra_Lobo_Logo, F.Cu at (114.5, 143.2)
