File: plusz-end-card-with-turnstile/plusz-end-card-with-turnstile.kicad_pcb (KiCad board)
At the start: 4 copper layers, 99.8 x 94.6 mm, 48 parts, among them J1 Harwin M55-7101242R, J10 R107064070_CONTACT, J11 R107064070_CONTACT, J12 R107064070_CONTACT, J13 R107064070_CONTACT, J14 R107064070_CONTACT, J15 R107064070_CONTACT, J16 R107064070_CONTACT, J2 Harwin M55-7101242R, J3 Harwin M55-7101242R, J4 Harwin M55-7101242R, J6 J-SAMTEC-TFM-120-X1-XXX-D-RA, J7 R107064070_CONTACT, J8 R107064070_CONTACT, J9 R107064070_CONTACT, U1 QCN-19+, U2 QCN-19+, U3 QCN-19+

Commit message: new
Parts:
- removed @HOLE0, @HOLE1, @HOLE2, @HOLE3: , 
- J10, J11, J12, J13, J14, J15, J16, J7, J8, J9: footprint plusz-end-card-with-turnstile:R107064070_CONTACT -> Foras_Promineo_Github_Local:R107064070_SOLDER
- J6: value J-SAMTEC-TFM-120-X1-XXX-D-RA -> (none)
Connections:
- net C3-UART-RX renamed /CONNECTORS/C3-UART-RX
- net C3-UART-TX renamed /CONNECTORS/C3-UART-TX
- net CAN1_H renamed /CONNECTORS/CAN1_H
- net CAN1_L renamed /CONNECTORS/CAN1_L
- net L1BAND_0 renamed /L1 BAND/L1BAND_0
- net L1BAND_180 renamed /L1 BAND/L1BAND_180
- net L1BAND_270 renamed /L1 BAND/L1BAND_270
- net L1BAND_90 renamed /L1 BAND/L1BAND_90
- net LBAND-1/4L renamed /L BAND/LBAND-1/4L
- net LBAND-SHORT renamed /L BAND/LBAND-SHORT
- net LBAND_0 renamed /L BAND/LBAND_0
- net LBAND_180 renamed /L BAND/LBAND_180
- net LBAND_270 renamed /L BAND/LBAND_270
- net LBAND_90 renamed /L BAND/LBAND_90
- net MAG-POWER renamed /CONNECTORS/MAG-POWER
- net MAG-SCL renamed /CONNECTORS/MAG-SCL
- net MAG-SDA renamed /CONNECTORS/MAG-SDA
- net TURNSTILE-DEPLOY renamed /CONNECTORS/TURNSTILE-DEPLOY
- net UHF_0 renamed /UHF/UHF_0
- net UHF_180 renamed /UHF/UHF_180
- net UHF_270 renamed /UHF/UHF_270
- net UHF_90 renamed /UHF/UHF_90
- net VBUS renamed /CONNECTORS/VBUS
- net ~{SD} renamed /CONNECTORS/~{SD}
- CF1 pad 10: (no net) -> unconnected-(CF1-Pad10)
- CF1 pad 11: (no net) -> unconnected-(CF1-Pad11)
- CF1 pad 12: (no net) -> unconnected-(CF1-Pad12)
- CF1 pad 9: (no net) -> unconnected-(CF1-Pad9)
- FIDUCIAL1 pad FIDUCIAL: (no net) -> unconnected-(FIDUCIAL1-PadFIDUCIAL)
- FIDUCIAL2 pad FIDUCIAL: (no net) -> unconnected-(FIDUCIAL2-PadFIDUCIAL)
- FIDUCIAL3 pad FIDUCIAL: (no net) -> unconnected-(FIDUCIAL3-PadFIDUCIAL)
- FIDUCIAL4 pad FIDUCIAL: (no net) -> unconnected-(FIDUCIAL4-PadFIDUCIAL)
- FIDUCIAL5 pad FIDUCIAL: (no net) -> unconnected-(FIDUCIAL5-PadFIDUCIAL)
- FIDUCIAL6 pad FIDUCIAL: (no net) -> unconnected-(FIDUCIAL6-PadFIDUCIAL)
- J12 pad P$1: L1BAND -> /L1 BAND/L1BAND
- J6 pad 11: (no net) -> unconnected-(J6-Pad11)
- J6 pad 12: (no net) -> unconnected-(J6-Pad12)
- J6 pad 13: (no net) -> unconnected-(J6-Pad13)
- J6 pad 14: (no net) -> unconnected-(J6-Pad14)
- J6 pad 15: (no net) -> unconnected-(J6-Pad15)
- J6 pad 16: (no net) -> unconnected-(J6-Pad16)
- J6 pad 17: (no net) -> unconnected-(J6-Pad17)
- J6 pad 18: (no net) -> unconnected-(J6-Pad18)
- J6 pad 19: (no net) -> unconnected-(J6-Pad19)
- J6 pad 20: (no net) -> unconnected-(J6-Pad20)
- J6 pad 21: (no net) -> unconnected-(J6-Pad21)
- J6 pad 22: (no net) -> unconnected-(J6-Pad22)
- J6 pad 31: (no net) -> unconnected-(J6-Pad31)
- J6 pad 32: (no net) -> unconnected-(J6-Pad32)
- J6 pad 7: (no net) -> unconnected-(J6-Pad7)
- J6 pad 8: (no net) -> unconnected-(J6-Pad8)
- J7 pad P$1: UHF -> /UHF/UHF
- U1 pad 1: LBAND -> /L BAND/LBAND
Routing:
- net LBAND: track 50.4 -> 0.00 mm, vias 1 -> 0
- net /L BAND/LBAND: track 0.00 -> 50.4 mm, vias 0 -> 1
- net L1BAND: track 19.0 -> 0.00 mm, vias 1 -> 0
- net /L1 BAND/L1BAND: track 0.00 -> 19.0 mm, vias 0 -> 1
- net UHF: track 11.7 -> 0.00 mm, vias 1 -> 0
- net /UHF/UHF: track 0.00 -> 11.7 mm, vias 0 -> 1
